File: Eagle/fonte12.brd (EAGLE design)
At the start: 100 x 80 mm, 12 parts, among them Q1 BC547B

Commit message: Atualização
Atualizei os arquivos do circuito, uma vez que precisei trocar o modelo do potenciômetro.
Parts:
- R2: value 5kΩ - 25mA -> 5kΩ; device pot:B64Y -> pot:3RP/1610N
- moved LED1 12.7 mm to (94.0, 11.4)
- moved R5 12.7 mm to (95.2, 24.1)
- moved Q1 11.4 mm to (84.2, 59.4)
- moved R4 10.2 mm to (85.1, 24.1)
- moved R1 5.08 mm to (52.1, 53.3)
- moved R2 2.54 mm to (63.5, 41.9)
Connections:
- net N$1: now also R2.1; no longer R2.A
- net N$12: now also R2.2; no longer R2.S
- net N$9: now also R2.3; no longer R2.E
Routing:
- net N$8: track 75.8 -> 120.5 mm
- net N$7: track 118.6 -> 95.9 mm
- net N$1: track 19.6 -> 6.43 mm
- net N$9: track 47.8 -> 36.9 mm
- net N$6: track 11.4 -> 21.6 mm
- net N$12: track 18.5 -> 27.2 mm
- net N$3: track 32.1 -> 39.7 mm
- net N$4: track 16.4 -> 14.9 mm

Commit message: Ajustes pós-apresentação
Adicionou-se a saída do sistema no lugar do R4
Parts:
- removed R4: 120Ω, rcl:0309/12
- added JP1: (no value), jumper:JP1
Connections:
- net N$3: now also JP1.2; no longer R4.1
- net N$6: no longer R4.2
- net N$8: now also JP1.1
Routing:
- net N$6: track 21.6 -> 0.00 mm
- net N$3: track 39.7 -> 53.7 mm
- net N$8: track 120.5 -> 131.3 mm
Changed lines of the file:
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@@
 <param name="PrefDir.14" value="0"/>
 <param name="PrefDir.15" value="0"/>
-<param name="PrefDir.16" value="-"/>
+<param name="PrefDir.16" value="a"/>
 <param name="cfVia" value="8"/>
 <param name="cfNonPref" value="5"/>
@@
 <attribute name="VALUE" x="64.1858" y="20.955" size="1.27" layer="27" ratio="10" rot="R90"/>
 </element>
-<element name="R4" library="rcl" library_urn="urn:adsk.eagle:library:334" package="0309/12" package3d_urn="urn:adsk.eagle:package:23571/1" value="120Ω" x="85.09" y="24.13" smashed="yes" rot="R270">
-<attribute name="NAME" x="86.995" y="28.321" size="1.27" layer="25" ratio="10" rot="R270"/>
-<attribute name="POPULARITY" value="8" x="45.72" y="3.81" size="1.778" layer="27" rot="R270" display="off"/>
-<attribute name="SPICEPREFIX" value="R" x="45.72" y="3.81" size="1.778" layer="27" rot="R270" display="off"/>
-<attribute name="VALUE" x="84.4042" y="27.305" size="1.27" layer="27" ratio="10" rot="R270"/>
-</element>
 <element name="R5" library="rcl" library_urn="urn:adsk.eagle:library:334" package="0309/12" package3d_urn="urn:adsk.eagle:package:23571/1" value="" x="95.25" y="24.13" smashed="yes" rot="R90">
 <attribute name="NAME" x="93.345" y="19.939" size="1.27" layer="26" ratio="10" rot="MR90"/>
@@
 <attribute name="POPULARITY" value="8" x="63.5" y="41.91" size="1.778" layer="27" rot="R90" display="off"/>
 <attribute name="VALUE" x="60.96" y="38.735" size="1.27" layer="27" rot="R90"/>
+</element>
+<element name="JP1" library="jumper" library_urn="urn:adsk.eagle:library:252" package="JP1" package3d_urn="urn:adsk.eagle:package:15455/1" value="" x="73.66" y="22.86" smashed="yes" rot="MR0">
+<attribute name="NAME" x="75.311" y="20.32" size="1.27" layer="25" ratio="10" rot="R90"/>
+<attribute name="POPULARITY" value="61" x="73.66" y="22.86" size="1.778" layer="28" rot="MR0" display="off"/>
+<attribute name="VALUE" x="70.739" y="20.32" size="1.27" layer="28" ratio="10" rot="MR90"/>
 </element>
 </elements>
@@
 <contactref element="D1" pad="A"/>
 <contactref element="LED1" pad="K"/>
-<wire x1="52.07" y1="11.43" x2="92.71" y2="11.43" width="1.016" layer="16"/>
+<wire x1="52.07" y1="11.43" x2="74.168" y2="11.43" width="1.016" layer="16"/>
+<wire x1="74.168" y1="11.43" x2="92.71" y2="11.43" width="1.016" layer="16"/>
 <wire x1="27.94" y1="31.75" x2="39.37" y2="43.18" width="1.016" layer="16"/>
 <wire x1="27.94" y1="6.6675" x2="27.94" y2="31.75" width="1.016" layer="16"/>
@@
 <wire x1="49.53" y1="8.89" x2="44.45" y2="13.97" width="1.016" layer="16"/>
 <wire x1="40.3225" y1="11.43" x2="40.132" y2="11.43" width="1.016" layer="16"/>
+<contactref element="JP1" pad="1"/>
+<wire x1="74.168" y1="11.43" x2="74.168" y2="21.336" width="1.016" layer="16"/>
+<wire x1="74.168" y1="21.336" x2="73.66" y2="21.59" width="1.016" layer="16"/>
+<wire x1="74.168" y1="11.176" x2="74.168" y2="11.43" width="1.016" layer="16"/>
 </signal>
 <signal name="N$9">
@@
 <signal name="N$3">
 <contactref element="Q1" pad="1"/>
-<contactref element="R4" pad="1"/>
 <contactref element="R5" pad="2"/>
 <wire x1="95.25" y1="30.48" x2="86.6775" y2="30.48" width="1.016" layer="16"/>
-<wire x1="86.6775" y1="30.48" x2="85.09" y2="30.48" width="1.016" layer="16"/>
 <wire x1="86.6775" y1="58.42" x2="85.725" y2="59.3725" width="1.016" layer="16"/>
 <wire x1="86.6775" y1="30.48" x2="86.6775" y2="58.42" width="1.016" layer="16"/>
 <wire x1="85.725" y1="59.3725" x2="85.471" y2="59.436" width="1.016" layer="16"/>
+<contactref element="JP1" pad="2"/>
+<wire x1="80.264" y1="24.384" x2="74.168" y2="24.384" width="1.016" layer="16"/>
+<wire x1="86.36" y1="30.48" x2="80.264" y2="24.384" width="1.016" layer="16"/>
+<wire x1="74.168" y1="24.384" x2="73.66" y2="24.13" width="1.016" layer="16"/>
+<wire x1="86.36" y1="30.48" x2="86.6775" y2="30.48" width="1.016" layer="16"/>
 </signal>
 <signal name="N$6">
-<contactref element="R4" pad="2"/>
 <contactref element="R3" pad="1"/>
-<wire x1="85.09" y1="17.78" x2="63.5" y2="17.78" width="1.016" layer="16"/>
 </signal>
 <signal name="N$10">
@@
 <wire x1="63.5" y1="41.91" x2="68.58" y2="41.91" width="1.016" layer="16"/>
 </signal>
+<signal name="N$14">
+</signal>
 </signals>
